File: LED-Board/LED-Board.kicad_sch (KiCad schematic)
At the start: 9 parts, among them J1 Header, Q1 NMOS, U1 IRS44273

Commit message: Continued Background
Parts:
- R1: value 20 -> R
Other:
- moved on the sheet: C1, C2, C3, C4, D1, J1, Q1, R1, U1

Commit message: Updated PCB
Parts:
- D1: footprint (none) -> IA-lib:JB3030
Connections:
- net GND: now also Q1.2 (S); no longer Q1.3 (S)
- net Gate: now also Q1.1 (G); no longer Q1.2 (G)
- net Drain: now reaches D1.1 (K)
- net Drain: now also Q1.3 (D); no longer Q1.1 (D)
Other:
- note removed: "TODO: Change NMOS footprint pins"
Changed lines of the file:
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@@
     (effects (font (size 2 2) (thickness 0.254) bold) (justify left bottom))
   )
-  (text "TODO: Change NMOS footprint pins" (at 58.42 180.34 0)
-    (effects (font (size 4 4) (thickness 0.8) bold (color 255 0 13 1)) (justify left bottom))
+  (label "Drain" (at 176.53 71.12 180) (fields_autoplaced)
+    (effects (font (size 1.27 1.27)) (justify right bottom))
   )
   (label "IN" (at 137.16 77.47 0) (fields_autoplaced)
@@
       (effects (font (size 1.27 1.27)) (justify right))
     )
-    (property "Footprint" "" (at 176.53 66.04 0)
-      (effects (font (size 1.27 1.27)) hide)
-    )
+    (property "Footprint" "IA-lib:JB3030" (at 176.53 66.04 0)
+      (effects (font (size 1.27 1.27)) hide)
+    )

Commit message: Appendix
Parts:
- C1, C2, C3, C4: value 22u -> 10u
- R1: value R -> 50
Connections:
- net +5V renamed VDC
